File: PCB/GB-Dumper.kicad_sch (KiCad schematic)
At the start: 18 parts, among them J1 GameBoy_Cartridge_MountingPin, J2 Conn_01x03_Pin, J3 Conn_01x03_Pin, J4 Conn_01x04_Pin, J5 Conn_01x03_Pin, J7 Conn_01x06_Pin, SW1 SW_SPDT, U1 SN74HC595_sorted, U2 SN74HC595_sorted

Commit message: cleanup
Connections:
- net GND: now also U2.13 (~{OE}), U2.8 (GND); no longer U2.16 (VCC), U2.5 (QF)
- net at A1.17 (+3V3), J7.6 (Pin_6), R1.2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: now also U2.10 (~{SRCLR}), U2.16 (VCC); no longer U2.2 (QC), U2.8 (GND)
- net at A1.16 (D13/PB5/SCK), J5.3 (Pin_3), J7.3 (Pin_3)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: now also U2.11 (SRCLK); no longer U2.3 (QD)
- net at A1.13 (D10/PB2/SS), J7.5 (Pin_5), U1.12 (RCLK): now also U2.12 (RCLK); no longer U2.4 (QE)
- net at U1.14 (SER): now also U2.9 (QH'); no longer U2.1 (QB)
- net at J1.10 (A4): now also U2.4 (QE); no longer U2.12 (RCLK)
- net at J1.11 (A5): now also U2.5 (QF); no longer U2.13 (~{OE})
- net at U2.14 (SER): now also A1.14 (D11/PB3/MOSI), J7.4 (Pin_4); no longer J1.12 (A6)
- net at U2.15 (QA): now also J1.6 (A0); no longer J1.13 (A7)
- net at U2.7 (QH): now also J1.13 (A7); no longer J1.6 (A0)
- net at J1.7 (A1): now also U2.1 (QB); no longer U2.9 (QH')
- net at J1.8 (A2): now also U2.2 (QC); no longer U2.10 (~{SRCLR})
- net at J1.9 (A3): now also U2.3 (QD); no longer U2.11 (SRCLK)
- new net: J1.12 (A6), U2.6 (QG)
- now unconnected: A1.14 (D11/PB3/MOSI)
Other:
- note added: "VIN/AUD(analog A1-5th sound-ch GB)=IRQ(D12 GBA)"
- note removed: "VIN(analog A1-5th sound-ch GB)=IRQ(D12 GBA)"
- moved on the sheet: TP1
Changed lines of the file:
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@@
 	(wire
 		(pts
-			(xy 69.85 113.03) (xy 69.85 119.38)
+			(xy 63.5 113.03) (xy 63.5 119.38)
 		)
 		(stroke
@@
 	(wire
 		(pts
-			(xy 69.85 113.03) (xy 86.36 113.03)
+			(xy 63.5 113.03) (xy 86.36 113.03)
 		)
 		(stroke
@@
 		)
 	)
-	(text "VIN(analog A1-5th sound-ch GB)=IRQ(D12 GBA)"
+	(text "VIN/AUD(analog A1-5th sound-ch GB)=IRQ(D12 GBA)"
 		(exclude_from_sim no)
 		(at 229.87 115.57 0)
@@
 	(text "I2C(RTC/Disp)"
 		(exclude_from_sim no)
-		(at 75.438 120.142 90)
+		(at 70.866 116.332 0)
 		(effects
 			(font
@@
 	(symbol
 		(lib_id "Connector:TestPoint")
-		(at 69.85 119.38 180)
+		(at 63.5 119.38 180)
 		(unit 1)
 		(exclude_from_sim no)
@@
 		(dnp no)
 		(property "Reference" "TP1"
-			(at 69.85 120.904 0)
+			(at 62.484 121.412 0)
 			(effects
 				(font
@@
 		)
 		(property "Value" "TestPoint"
-			(at 68.834 118.872 0)
+			(at 72.644 121.412 0)
 			(effects
 				(font
@@
 		)
 		(property "Footprint" "TestPoint:TestPoint_THTPad_2.5x2.5mm_Drill1.2mm"
-			(at 61.976 147.32 90)
+			(at 55.626 147.32 90)
 			(effects
 				(font
@@
 		)
 		(property "Datasheet" "~"
-			(at 64.77 119.38 0)
+			(at 58.42 119.38 0)
 			(effects
 				(font
@@
 		)
 		(property "Description" ""
-			(at 69.85 119.38 0)
+			(at 63.5 119.38 0)
 			(effects
 				(font
@@
 	)
 	(symbol
+		(lib_id "SN74HC595_sorted:74HC595_sorted")
+		(at 123.19 62.23 180)
+		(unit 1)
+		(exclude_from_sim no)
+		(in_bom yes)
+		(on_board yes)
+		(dnp no)
+		(property "Reference" "U2"
+			(at 132.588 73.406 0)
+			(effects
+				(font
+					(size 1.27 1.27)
+				)
+			)
+		)
+		(property "Value" "SN74HC595_sorted"
+			(at 123.19 44.45 0)
+			(effects
+				(font
+					(size 1.27 1.27)
+				)
+			)
+		)
+		(property "Footprint" "Gameboy_THT:SN74HC595"
+			(at 123.19 62.23 0)
+			(effects
+				(font
+					(size 1.27 1.27)
+				)
+				(hide yes)
+			)
+		)
+		(property "Datasheet" "http://www.ti.com/lit/ds/symlink/sn74hc595.pdf"
+			(at 93.98 71.12 90)
+			(effects
+				(font
+					(size 1.27 1.27)
+				)
+				(hide yes)
+			)
+		)
+		(property "Description" ""
+			(at 123.19 62.23 0)
+			(effects
+				(font
+					(size 1.27 1.27)
+				)
+				(hide yes)
+			)
+		)
+		(pin "7"
+		)
+		(pin "5"
+		)
+		(pin "10"
+		)
+		(pin "14"
+		)
+		(pin "4"
+		)
+		(pin "15"
+		)
+		(pin "16"
+		)
+		(pin "8"
+		)
+		(pin "11"
+		)
+		(pin "2"
+		)
+		(pin "6"
+		)
+		(pin "12"
+		)
+		(pin "13"
+		)
+		(pin "3"
+		)
+		(pin "1"
+		)
+		(pin "9"
+		)
+		(instances
+			(project "GB-Dumper"
+				(path "/20f6159f-fd4e-4dc1-b76c-f4f6e70e964a"
+					(reference "U2")
+					(unit 1)
+				)
+			)
+		)
+	)
+	(symbol
 		(lib_id "Connector:Conn_01x06_Pin")
 		(at 53.34 38.1 0)
@@
 					(unit 1)
 				)
-			)
-		)
-	)
-	(symbol
-		(lib_id "SN74HC595_sorted:74HC595_sorted")
-		(at 123.19 59.69 0)
-		(unit 1)
-		(exclude_from_sim no)
-		(in_bom yes)
-		(on_board yes)
-		(dnp no)
-		(property "Reference" "U2"
-			(at 113.792 48.514 0)
-			(effects
-				(font
-					(size 1.27 1.27)
-				)
-			)
-		)
-		(property "Value" "SN74HC595_sorted"
-			(at 123.19 77.47 0)
-			(effects
-				(font
-					(size 1.27 1.27)
-				)
-			)
-		)
-		(property "Footprint" "Gameboy_THT:SN74HC595"
-			(at 123.19 59.69 0)
-			(effects
-				(font
-					(size 1.27 1.27)
-				)
-				(hide yes)
-			)
-		)
-		(property "Datasheet" "http://www.ti.com/lit/ds/symlink/sn74hc595.pdf"
-			(at 152.4 50.8 90)
-			(effects
-				(font
-					(size 1.27 1.27)
-				)
-				(hide yes)
-			)
-		)
-		(property "Description" ""
-			(at 123.19 59.69 0)
-			(effects
-				(font
-					(size 1.27 1.27)
-				)
-				(hide yes)
-			)
-		)
-		(pin "7"
-		)
-		(pin "5"
-		)
-		(pin "10"
-		)
-		(pin "14"
-		)
-		(pin "4"
-		)
-		(pin "15"
-		)
-		(pin "16"
-		)
-		(pin "8"
-		)
-		(pin "11"
-		)
-		(pin "2"
-		)
-		(pin "6"
-		)
-		(pin "12"
-		)
-		(pin "13"
-		)
-		(pin "3"
-		)
-		(pin "1"
-		)
-		(pin "9"
-		)
-		(instances
-			(project "GB-Dumper"
-				(path "/20f6159f-fd4e-4dc1-b76c-f4f6e70e964a"
-					(reference "U2")
-					(unit 1)
-				)
